File: hardware/encoder.kicad_sch (KiCad schematic)
At the start: 6 parts, among them SW57 RotaryEncoder_Switch_MP

Commit message: electronics
Parts:
- C36: renamed from C75; footprint PCM_Capacitor_SMD_AKL:C_0603_1608Metric -> PCM_Capacitor_SMD_Handsoldering_AKL:C_0603_1608Metric; Distributor Link 3 (none) -> https://www.hestore.hu/prod_10033461.html
- C37: renamed from C76; footprint PCM_Capacitor_SMD_AKL:C_0603_1608Metric -> PCM_Capacitor_SMD_Handsoldering_AKL:C_0603_1608Metric; Distributor Link 3 (none) -> https://www.hestore.hu/prod_10033461.html
- R19: renamed from R41; footprint PCM_Resistor_SMD_AKL:R_0603_1608Metric_Pad0.98x0.95mm_HandSolder -> PCM_Resistor_SMD_AKL:R_0603_1608Metric; Distributor Link 3 (none) -> https://www.hestore.hu/prod_10023910.html
- R20: renamed from R40; footprint PCM_Resistor_SMD_AKL:R_0603_1608Metric_Pad0.98x0.95mm_HandSolder -> PCM_Resistor_SMD_AKL:R_0603_1608Metric; Distributor Link 3 (none) -> https://www.hestore.hu/prod_10023910.html
- SW29: renamed from SW57; footprint Rotary_Encoder:RotaryEncoder_Alps_EC11E-Switch_Vertical_H20mm -> rp_voyager:RotaryEncoder_Alps_EC11S-Switch_Vertical_H9mm
- renumbered D114 to D57
Changed lines of the file:
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@@
 		(dnp no)
 		(fields_autoplaced yes)
-		(property "Reference" "#PWR048"
+		(property "Reference" "#PWR070"
 			(at 132.08 115.57 0)
 			(hide yes)
@@
 			(project "rp_voyager"
 				(path "/16aaafff-4e4d-4193-9340-05bf864eda5e/9ca86edd-3683-462d-b98a-f0d936a65f5b/22a0881f-8879-456d-b0b2-3f3994f164ed"
-					(reference "#PWR048")
+					(reference "#PWR0144")
 					(unit 1)
 				)
 				(path "/16aaafff-4e4d-4193-9340-05bf864eda5e/c41eb395-0a81-4295-aa13-94d2d2590030/48194633-b25b-4431-875c-e0dd69517d2a"
-					(reference "#PWR048")
+					(reference "#PWR070")
 					(unit 1)
 				)
@@
 		(in_pos_files yes)
 		(dnp no)
-		(property "Reference" "SW57"
+		(property "Reference" "SW29"
 			(at 153.67 72.39 90)
 			(show_name no)
@@
 			)
 		)
-		(property "Footprint" "Rotary_Encoder:RotaryEncoder_Alps_EC11E-Switch_Vertical_H20mm"
+		(property "Footprint" "rp_voyager:RotaryEncoder_Alps_EC11S-Switch_Vertical_H9mm"
 			(at 149.606 92.71 0)
 			(hide yes)
@@
 		(property "Description" "Rotary encoder, dual channel, incremental quadrate outputs, with switch and MP Pin"
 			(at 168.91 88.9 0)
+			(hide yes)
+			(show_name no)
+			(do_not_autoplace no)
+			(effects
+				(font
+					(size 1.27 1.27)
+				)
+			)
+		)
+		(property "Manufacturer" ""
+			(at 153.67 88.9 0)
+			(hide yes)
+			(show_name no)
+			(do_not_autoplace no)
+			(effects
+				(font
+					(size 1.27 1.27)
+				)
+			)
+		)
+		(property "Distributor Link 1" ""
+			(at 153.67 88.9 0)
+			(hide yes)
+			(show_name no)
+			(do_not_autoplace no)
+			(effects
+				(font
+					(size 1.27 1.27)
+				)
+			)
+		)
+		(property "Distributor Link 2" ""
+			(at 153.67 88.9 0)
+			(hide yes)
+			(show_name no)
+			(do_not_autoplace no)
+			(effects
+				(font
+					(size 1.27 1.27)
+				)
+			)
+		)
+		(property "Distributor Link 3" ""
+			(at 153.67 88.9 0)
 			(hide yes)
 			(show_name no)
@@
 				)
 				(path "/16aaafff-4e4d-4193-9340-05bf864eda5e/c41eb395-0a81-4295-aa13-94d2d2590030/48194633-b25b-4431-875c-e0dd69517d2a"
-					(reference "SW57")
+					(reference "SW29")
 					(unit 1)
 				)
@@
 		(dnp no)
 		(fields_autoplaced yes)
-		(property "Reference" "#PWR046"
+		(property "Reference" "#PWR072"
 			(at 161.29 95.25 0)
 			(hide yes)
@@
 			(project "rp_voyager"
 				(path "/16aaafff-4e4d-4193-9340-05bf864eda5e/9ca86edd-3683-462d-b98a-f0d936a65f5b/22a0881f-8879-456d-b0b2-3f3994f164ed"
-					(reference "#PWR046")
+					(reference "#PWR0146")
 					(unit 1)
 				)
 				(path "/16aaafff-4e4d-4193-9340-05bf864eda5e/c41eb395-0a81-4295-aa13-94d2d2590030/48194633-b25b-4431-875c-e0dd69517d2a"
-					(reference "#PWR046")
+					(reference "#PWR072")
 					(unit 1)
 				)
@@
 		(dnp no)
 		(fields_autoplaced yes)
-		(property "Reference" "D114"
+		(property "Reference" "D57"
 			(at 172.72 69.85 0)
 			(show_name no)
@@
 				)
 				(path "/16aaafff-4e4d-4193-9340-05bf864eda5e/c41eb395-0a81-4295-aa13-94d2d2590030/48194633-b25b-4431-875c-e0dd69517d2a"
-					(reference "D114")
+					(reference "D57")
 					(unit 1)
 				)
@@
 		(dnp no)
 		(fields_autoplaced yes)
-		(property "Reference" "#PWR044"
+		(property "Reference" "#PWR071"
 			(at 153.67 107.95 0)
 			(hide yes)
@@
 			(project "rp_voyager"
 				(path "/16aaafff-4e4d-4193-9340-05bf864eda5e/9ca86edd-3683-462d-b98a-f0d936a65f5b/22a0881f-8879-456d-b0b2-3f3994f164ed"
-					(reference "#PWR044")
+					(reference "#PWR0145")
 					(unit 1)
 				)
 				(path "/16aaafff-4e4d-4193-9340-05bf864eda5e/c41eb395-0a81-4295-aa13-94d2d2590030/48194633-b25b-4431-875c-e0dd69517d2a"
-					(reference "#PWR044")
+					(reference "#PWR071")
 					(unit 1)
 				)
@@
 		(dnp no)
 		(fields_autoplaced yes)
-		(property "Reference" "R40"
+		(property "Reference" "R20"
 			(at 172.72 96.5199 0)
 			(show_name no)
@@
 			)
 		)
-		(property "Footprint" "PCM_Resistor_SMD_AKL:R_0603_1608Metric_Pad0.98x0.95mm_HandSolder"
+		(property "Footprint" "PCM_Resistor_SMD_AKL:R_0603_1608Metric"
 			(at 170.18 97.79 0)
 			(hide yes)
@@
 			)
 		)
-		(property "Distributor Link 3" ""
+		(property "Distributor Link 3" "https://www.hestore.hu/prod_10023910.html"
 			(at 170.18 97.79 0)
 			(hide yes)
@@
 			(project "rp_voyager"
 				(path "/16aaafff-4e4d-4193-9340-05bf864eda5e/9ca86edd-3683-462d-b98a-f0d936a65f5b/22a0881f-8879-456d-b0b2-3f3994f164ed"
-					(reference "R17")
+					(reference "R41")
 					(unit 1)
 				)
 				(path "/16aaafff-4e4d-4193-9340-05bf864eda5e/c41eb395-0a81-4295-aa13-94d2d2590030/48194633-b25b-4431-875c-e0dd69517d2a"
-					(reference "R40")
+					(reference "R20")
 					(unit 1)
 				)
@@
 		(in_pos_files yes)
 		(dnp no)
-		(property "Reference" "C76"
+		(property "Reference" "C37"
 			(at 172.72 105.4162 0)
 			(show_name no)
@@
 			)
 		)
-		(property "Footprint" "PCM_Capacitor_SMD_AKL:C_0603_1608Metric"
+		(property "Footprint" "PCM_Capacitor_SMD_Handsoldering_AKL:C_0603_1608Metric"
 			(at 170.18 106.68 0)
 			(hide yes)
@@
 			)
 		)
-		(property "Distributor Link 3" ""
+		(property "Distributor Link 3" "https://www.hestore.hu/prod_10033461.html"
 			(at 170.18 106.68 0)
 			(hide yes)
@@
 			(project "rp_voyager"
 				(path "/16aaafff-4e4d-4193-9340-05bf864eda5e/9ca86edd-3683-462d-b98a-f0d936a65f5b/22a0881f-8879-456d-b0b2-3f3994f164ed"
-					(reference "C78")
+					(reference "C74")
 					(unit 1)
 				)
 				(path "/16aaafff-4e4d-4193-9340-05bf864eda5e/c41eb395-0a81-4295-aa13-94d2d2590030/48194633-b25b-4431-875c-e0dd69517d2a"
-					(reference "C76")
+					(reference "C37")
 					(unit 1)
 				)
@@
 		(in_pos_files yes)
 		(dnp no)
-		(property "Reference" "C75"
+		(property "Reference" "C36"
 			(at 134.62 105.4162 0)
 			(show_name no)
@@
 			)
 		)
-		(property "Footprint" "PCM_Capacitor_SMD_AKL:C_0603_1608Metric"
+		(property "Footprint" "PCM_Capacitor_SMD_Handsoldering_AKL:C_0603_1608Metric"
 			(at 132.08 106.68 0)
 			(hide yes)
@@
 			)
 		)
-		(property "Distributor Link 3" ""
+		(property "Distributor Link 3" "https://www.hestore.hu/prod_10033461.html"
 			(at 132.08 106.68 0)
 			(hide yes)
@@
 			(project "rp_voyager"
 				(path "/16aaafff-4e4d-4193-9340-05bf864eda5e/9ca86edd-3683-462d-b98a-f0d936a65f5b/22a0881f-8879-456d-b0b2-3f3994f164ed"
-					(reference "C77")
+					(reference "C73")
 					(unit 1)
 				)
 				(path "/16aaafff-4e4d-4193-9340-05bf864eda5e/c41eb395-0a81-4295-aa13-94d2d2590030/48194633-b25b-4431-875c-e0dd69517d2a"
-					(reference "C75")
+					(reference "C36")
 					(unit 1)
 				)
@@
 		(dnp no)
 		(fields_autoplaced yes)
-		(property "Reference" "R41"
+		(property "Reference" "R19"
 			(at 134.62 96.5199 0)
 			(show_name no)
@@
 			)
 		)
-		(property "Footprint" "PCM_Resistor_SMD_AKL:R_0603_1608Metric_Pad0.98x0.95mm_HandSolder"
+		(property "Footprint" "PCM_Resistor_SMD_AKL:R_0603_1608Metric"
 			(at 132.08 97.79 0)
 			(hide yes)
@@
 			)
 		)
-		(property "Distributor Link 3" ""
+		(property "Distributor Link 3" "https://www.hestore.hu/prod_10023910.html"
 			(at 132.08 97.79 0)
 			(hide yes)
@@
 			(project "rp_voyager"
 				(path "/16aaafff-4e4d-4193-9340-05bf864eda5e/9ca86edd-3683-462d-b98a-f0d936a65f5b/22a0881f-8879-456d-b0b2-3f3994f164ed"
-					(reference "R14")
+					(reference "R40")
 					(unit 1)
 				)
 				(path "/16aaafff-4e4d-4193-9340-05bf864eda5e/c41eb395-0a81-4295-aa13-94d2d2590030/48194633-b25b-4431-875c-e0dd69517d2a"
-					(reference "R41")
+					(reference "R19")
 					(unit 1)
 				)
@@
 		(dnp no)
 		(fields_autoplaced yes)
-		(property "Reference" "#PWR0116"
+		(property "Reference" "#PWR073"
 			(at 170.18 115.57 0)
 			(hide yes)
@@
 			(project "rp_voyager"
 				(path "/16aaafff-4e4d-4193-9340-05bf864eda5e/9ca86edd-3683-462d-b98a-f0d936a65f5b/22a0881f-8879-456d-b0b2-3f3994f164ed"
-					(reference "#PWR0116")
+					(reference "#PWR0147")
 					(unit 1)
 				)
 				(path "/16aaafff-4e4d-4193-9340-05bf864eda5e/c41eb395-0a81-4295-aa13-94d2d2590030/48194633-b25b-4431-875c-e0dd69517d2a"
-					(reference "#PWR0116")
-					(unit 1)
-				)
+					(reference "#PWR073")
+					(unit 1)
+				)
