File: hardware/usbc.kicad_sch (KiCad schematic)
At the start: 18 parts, among them J1 INPUT USB, U1 TPS259261, U2 AP2125N-3.3TRG1

Commit message: encoder to schematic
Parts:
- added C25: 10n, PCM_Capacitor_SMD_AKL:C_0603_1608Metric_Pad1.05x0.95mm_HandSolder, symbol Device:C_Small
- added C26: 220u, PCM_Capacitor_SMD_AKL:C_1210_3225Metric_Pad1.33x2.70mm_HandSolder, symbol Device:C_Small
- added C27: 100n, PCM_Capacitor_SMD_AKL:C_0603_1608Metric, symbol Device:C_Small
- added D28, D30: DESD5V0U1BA-7, PCM_Diode_SMD_AKL:D_SOD-323_HandSoldering, symbol PCM_Diode_TVS_AKL:D_TVS_Bidirectional_Generic
- added D29: SZSMF5.0AT1G, PCM_Diode_SMD_Handsoldering_AKL:D_SOD-123_TVS, symbol PCM_Diode_TVS_AKL:D_TVS_Unidirectional_Generic
- added J2: UART USB, Connector_USB:USB_C_Receptacle_GCT_USB4105-xx-A_16P_TopMnt_Horizontal, symbol Connector:USB_C_Receptacle_USB2.0_14P
- added JP1: No shunt, Jumper:SolderJumper-2_P1.3mm_Bridged_RoundedPad1.0x1.5mm, symbol Jumper:SolderJumper_2_Bridged
- added R12, R13: 5.1k, PCM_Resistor_SMD_AKL:R_0603_1608Metric_Pad0.98x0.95mm_HandSolder, symbol Device:R_Small
- added R15, R18: 220, PCM_Resistor_SMD_AKL:R_0603_1608Metric_Pad0.98x0.95mm_HandSolder, symbol Device:R_Small
- added R16: 0, PCM_Resistor_SMD_AKL:R_1206_3216Metric_Pad1.30x1.75mm_HandSolder, symbol Device:R_Small
- added TP1: UART_TX, TestPoint:TestPoint_Pad_D2.0mm, symbol Connector:TestPoint
- added TP2: I2C 5V, TestPoint:TestPoint_Pad_D2.0mm, symbol Connector:TestPoint
- added TP3: UART_RX, TestPoint:TestPoint_Pad_D2.0mm, symbol Connector:TestPoint
Connections:
- net +5V: now also C26.1, C27.1, JP1.2 (B), R16.1
- net GND: now also C25.2, C26.2, C27.2, D28.1 (K), D29.2 (A), D30.1 (K), J2.A1 (GND), J2.A12 (GND), J2.B1 (GND), J2.B12 (GND), J2.SH (SHIELD), R12.2, R13.2
- new net CONN_CC1: J2.A5 (CC1), R12.1
- new net CONN_CC2: J2.B5 (CC2), R13.1
- new net CONN_RX: D30.2 (A), J2.A7 (D-), J2.B7 (D-), R18.1, TP3.1
- new net CONN_TX: D28.2 (A), J2.A6 (D+), J2.B6 (D+), R15.1, TP1.1
- new net CONN_VBUS: C25.1, D29.1 (K), J2.A4 (VBUS), J2.A9 (VBUS), J2.B4 (VBUS), J2.B9 (VBUS), JP1.1 (A), R16.2, TP2.1
- new net UART_RX: R18.2
- new net UART_TX: R15.2
Other:
- moved on the sheet: C1, C2, C3, C4, C5, C6, C7, C8, C9, D1, J1, R1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

Commit message: electronics
Parts:
- removed C26: 220u, PCM_Capacitor_SMD_AKL:C_1210_3225Metric_Pad1.33x2.70mm_HandSolder, symbol Device:C_Small
- removed C27: 100n, PCM_Capacitor_SMD_AKL:C_0603_1608Metric, symbol Device:C_Small
- C1: footprint PCM_Capacitor_SMD_AKL:C_0603_1608Metric_Pad1.05x0.95mm_HandSolder -> PCM_Capacitor_SMD_Handsoldering_AKL:C_0603_1608Metric; Distributor Link 3 (none) -> https://www.hestore.hu/prod_10033461.html
- C10: renamed from C6; footprint PCM_Capacitor_SMD_AKL:C_0805_2012Metric_Pad1.15x1.40mm_HandSolder -> PCM_Capacitor_SMD_Handsoldering_AKL:C_0805_2012Metric; Distributor Link 1 (none) -> https://hu.mouser.com/ProductDetail/KEMET/C0805C106M8RACAUT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
- C2: footprint PCM_Capacitor_SMD_AKL:C_0603_1608Metric_Pad1.05x0.95mm_HandSolder -> PCM_Capacitor_SMD_Handsoldering_AKL:C_0603_1608Metric; Distributor Link 3 (none) -> https://www.hestore.hu/prod_10043666.html
- C3: footprint PCM_Capacitor_SMD_AKL:C_0603_1608Metric_Pad1.05x0.95mm_HandSolder -> PCM_Capacitor_SMD_Handsoldering_AKL:C_0603_1608Metric; Distributor Link 3 (none) -> https://www.hestore.hu/prod_10027791.html
- C4: renamed from C25; footprint PCM_Capacitor_SMD_AKL:C_0603_1608Metric_Pad1.05x0.95mm_HandSolder -> PCM_Capacitor_SMD_Handsoldering_AKL:C_0603_1608Metric
- C5: renamed from C4; footprint PCM_Capacitor_SMD_AKL:C_0603_1608Metric_Pad1.05x0.95mm_HandSolder -> PCM_Capacitor_SMD_Handsoldering_AKL:C_0603_1608Metric
- C6: renamed from C7; footprint PCM_Capacitor_SMD_AKL:C_0603_1608Metric_Pad1.05x0.95mm_HandSolder -> PCM_Capacitor_SMD_Handsoldering_AKL:C_0603_1608Metric; Distributor Link 3 (none) -> https://www.hestore.hu/prod_10033461.html
- C7: renamed from C8; footprint PCM_Capacitor_SMD_AKL:C_1210_3225Metric_Pad1.33x2.70mm_HandSolder -> PCM_Capacitor_SMD_Handsoldering_AKL:C_1210_3225Metric; Distributor Link 1 (none) -> https://hu.mouser.com/ProductDetail/KYOCERA-AVX/TCJB227M006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
- C8: renamed from C9; footprint PCM_Capacitor_SMD_AKL:C_0805_2012Metric_Pad1.15x1.40mm_HandSolder -> PCM_Capacitor_SMD_Handsoldering_AKL:C_0805_2012Metric; Distributor Link 1 (none) -> https://hu.mouser.com/ProductDetail/KEMET/C0805C106M8RACAUT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
- C9: renamed from C5; footprint PCM_Capacitor_SMD_AKL:C_0603_1608Metric_Pad1.05x0.95mm_HandSolder -> PCM_Capacitor_SMD_Handsoldering_AKL:C_0603_1608Metric; Distributor Link 3 (none) -> https://www.hestore.hu/prod_10033461.html
- D1: renamed from D28; footprint PCM_Diode_SMD_AKL:D_SOD-323_HandSoldering -> PCM_Diode_SMD_Handsoldering_AKL:D_SOD-323_TVS
- D2: renamed from D1; value SR05 -> PRTR5V0U2X; Distributor Link 1 https://hu.mouser.com/ProductDetail/Micro-Commercial-Compon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 -> https://hu.mouser.com/ProductDetail/Nexperia/PRTR5V0U2X215?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
- D3: renamed from D29; footprint PCM_Diode_SMD_Handsoldering_AKL:D_SOD-123_TVS -> PCM_Diode_SMD_Handsoldering_AKL:D_SOD-123_Zener
- D4: renamed from D30; footprint PCM_Diode_SMD_AKL:D_SOD-323_HandSoldering -> PCM_Diode_SMD_Handsoldering_AKL:D_SOD-323_TVS
- R1: renamed from R15; footprint PCM_Resistor_SMD_AKL:R_0603_1608Metric_Pad0.98x0.95mm_HandSolder -> PCM_Resistor_SMD_AKL:R_0603_1608Metric; Distributor Link 3 (none) -> https://www.hestore.hu/prod_10036836.html
- R10: renamed from R5; footprint PCM_Resistor_SMD_AKL:R_0603_1608Metric_Pad0.98x0.95mm_HandSolder -> PCM_Resistor_SMD_AKL:R_0603_1608Metric; Distributor Link 3 (none) -> https://www.hestore.hu/prod_10043634.html
- R2: renamed from R1; footprint PCM_Resistor_SMD_AKL:R_0603_1608Metric_Pad0.98x0.95mm_HandSolder -> PCM_Resistor_SMD_AKL:R_0603_1608Metric; Distributor Link 3 (none) -> https://www.hestore.hu/prod_10036539.html
- R3: renamed from R2; footprint PCM_Resistor_SMD_AKL:R_0603_1608Metric_Pad0.98x0.95mm_HandSolder -> PCM_Resistor_SMD_AKL:R_0603_1608Metric; Distributor Link 3 (none) -> https://www.hestore.hu/prod_10036539.html
- R4: renamed from R12; footprint PCM_Resistor_SMD_AKL:R_0603_1608Metric_Pad0.98x0.95mm_HandSolder -> PCM_Resistor_SMD_AKL:R_0603_1608Metric; Distributor Link 3 (none) -> https://www.hestore.hu/prod_10036539.html
- R5: renamed from R13; footprint PCM_Resistor_SMD_AKL:R_0603_1608Metric_Pad0.98x0.95mm_HandSolder -> PCM_Resistor_SMD_AKL:R_0603_1608Metric; Distributor Link 3 (none) -> https://www.hestore.hu/prod_10036539.html
- R6: renamed from R18; footprint PCM_Resistor_SMD_AKL:R_0603_1608Metric_Pad0.98x0.95mm_HandSolder -> PCM_Resistor_SMD_AKL:R_0603_1608Metric; Distributor Link 3 (none) -> https://www.hestore.hu/prod_10036836.html
- R7: renamed from R3; Distributor Link 3 (none) -> https://www.hestore.hu/prod_10023910.html
- R8: renamed from R4; Distributor Link 3 (none) -> https://www.hestore.hu/prod_10043366.html
- R9: renamed from R16; footprint PCM_Resistor_SMD_AKL:R_1206_3216Metric_Pad1.30x1.75mm_HandSolder -> PCM_Resistor_SMD_AKL:R_1206_3216Metric
- renumbered TP3 to TP2, TP2 to TP3
Other:
- moved on the sheet: C10, C9, TP3, U2
