File: hardware/rp_voyager.kicad_pcb (KiCad board)
At the start: 4 copper layers, 150.5 x 141.7 mm, 317 parts, among them J1 INPUT USB, J2 UART USB, J3 INPUT USB, J4 UART USB, Q1 2N7002, SW1 RESET, SW10 Key, SW11 Key, SW12 Key, SW13 Key, SW14 Key, SW15 Key, SW16 Key, SW17 Key, SW18 Key, SW19 Key, SW2 BOOTSEL, SW20 Key, SW21 Key, SW22 Key, SW23 Key, SW24 Key, SW25 Key, SW26 Key, SW27 Key, SW28 Key, SW29 RotaryEncoder_Switch_MP, SW3 Key, SW30 RESET, SW31 BOOTSEL, SW32 Key, SW33 Key, SW34 Key, SW35 Key, SW36 Key, SW37 Key, SW38 Key, SW39 Key, SW4 Key, SW40 Key, SW41 Key, SW42 Key, SW43 Key, SW44 Key, SW45 Key, SW46 Key, SW47 Key, SW48 Key, SW49 Key, SW5 Key, SW50 Key, SW51 Key, SW52 Key, SW53 Key, SW54 Key, SW55 Key, SW56 Key, SW57 Key, SW58 RotaryEncoder_Switch_MP, SW6 Key, SW7 Key, SW8 Key, SW9 Key, U1 TPS259261, U2 AP2125N-3.3TRG1, U3 RP2354A, U4 74HCT1G125GW, U5 TPS259261, U6 AP2125N-3.3TRG1, U7 RP2354A, U8 74HCT1G125GW, Y1 12MHz, Y2 12MHz

Commit message: updated pcb to latest tray layout
Parts:
- added makersmark1: ~, rp_voyager:julian7_makers_mark, F.Cu at (84.6, 54.9)
- moved R21 10.7 mm to (218.2, 126.1), turned to 90 degrees
- moved R26 8.16 mm to (220.0, 126.1), turned to 90 degrees
- moved R25 4.07 mm to (225.2, 133.2)
- moved R24 2.87 mm to (220.4, 137.7)
- moved J3 2.84 mm to (224.1, 99.7)
- moved C65 2.82 mm to (248.1, 60.4)
- moved C69 2.82 mm to (248.1, 58.3)
- moved D60 2.79 mm to (222.0, 130.1)
- moved J4 2.78 mm to (214.5, 133.3)
- moved C59 2.77 mm to (222.2, 112.5)
- moved D107 2.77 mm to (330.2, 57.8)
- moved D110 2.77 mm to (330.2, 115.0)
- moved D111 2.77 mm to (349.2, 57.8)
- moved D114 2.77 mm to (349.2, 115.0)
- moved D65 2.77 mm to (353.7, 103.7)
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Routing:
- net (no net): track 19.6 -> 0.00 mm
- net /Right/Connector and Power/UART_TX: track 31.9 -> 16.8 mm
- net /Right/Connector and Power/UART_RX: track 27.0 -> 15.1 mm
- net Net-(D34-DIN): track 22.3 -> 29.6 mm, vias 2 -> 0
- net /Left/Key Matrix/COL1: track 179.4 -> 173.4 mm
- net Net-(D44-DIN): track 34.8 -> 29.8 mm
- net Net-(D52-DIN): track 36.6 -> 31.7 mm
- net /Right/Key Matrix (copy)/COL0: track 188.2 -> 183.4 mm
- net Net-(D48-DIN): track 34.6 -> 29.8 mm
- net Net-(D93-DOUT): track 18.8 -> 23.3 mm
- net /Right/Connector and Power/CONN_RX: track 12.3 -> 16.8 mm
- net Net-(D92-DOUT): track 53.9 -> 50.1 mm
- net /Right/Key Matrix (copy)/COL2: track 139.4 -> 143.0 mm
- net /Left/Backlight RGB LEDs/RGB_DATA: track 21.0 -> 18.6 mm
- net GND: track 259.9 -> 257.9 mm
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Other:
- outline, holes or cut-outs redrawn
- board text added: "Thank you ZSA Technology Labs, for the awesome design! https://www.zsa.io/voyager"

Commit message: JLCDFM check and renders
Routing:
- net GND: track 257.9 -> 252.0 mm
- net /Right/Connector and Power/USB_CC2: track 10.4 -> 6.98 mm
- net Net-(D62-A): track 33.7 -> 31.8 mm
- net /Right/Key Matrix (copy)/ROW1: track 162.6 -> 160.7 mm
- net /Right/Key Matrix (copy)/ROW0: track 182.2 -> 180.7 mm
- net /Left/Key Matrix/COL2: track 152.6 -> 151.6 mm
- net /Right/Connector and Power/USB_CC1: track 3.34 -> 4.27 mm
- net /Right/Connector and Power/+3.3V: track 84.7 -> 85.4 mm
- net Net-(U7-~{QSPI_SS}): track 46.3 -> 46.9 mm
- net /Left/Connector and Power/+3.3V: track 100.0 -> 100.5 mm
- net /Right/Connector and Power/VBUS: track 27.0 -> 27.5 mm
- net /Right/Encoder (copy)/SW_COL: track 196.4 -> 195.9 mm

Commit message: make the pcb compatible with kailh choc v1/v2
Parts:
- removed JP1, JP2: No shunt, Jumper:SolderJumper-2_P1.3mm_Bridged_RoundedPad1.0x1.5mm
- R29, R9: footprint PCM_Resistor_SMD_AKL:R_1206_3216Metric -> rp_voyager:R_1206_3216Metric_WireJumper
- moved C69 16.1 mm to (262.2, 50.5), turned to 90 degrees
- moved C65 15.6 mm to (260.1, 50.4), turned to 90 degrees
- moved C70 4.73 mm to (246.6, 71.7)
- moved C66 4.73 mm to (246.6, 74.0)
- moved R33 3.56 mm to (268.1, 107.1), turned to 180 degrees
- moved C68 3.52 mm to (246.1, 115.8)
- moved C72 3.39 mm to (246.4, 113.4)
- moved D19 2.29 mm to (128.4, 95.3)
- moved D27 2.28 mm to (166.5, 85.8)
- moved D24 2.24 mm to (147.5, 119.2)
- moved D26 2.24 mm to (166.5, 66.8)
- moved D12 2.03 mm to (90.3, 123.9)
- moved R34 2.01 mm to (268.1, 105.1), turned to 180 degrees
- moved D7 1.99 mm to (71.3, 104.9)
- moved D11 1.98 mm to (90.3, 104.9)
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Routing:
- net /Right/Connector and Power/+5V: track 617.3 -> 635.0 mm
- net /Left/Key Matrix/ROW2: track 118.4 -> 111.5 mm
- net Net-(D37-DIN): track 29.9 -> 36.8 mm
- net Net-(D102-DIN): track 36.0 -> 31.2 mm
- net GND: track 252.0 -> 256.6 mm, vias 238 -> 265
- net /Left/Key Matrix/COL0: track 195.0 -> 198.9 mm
- net Net-(R33-Pad2): track 1.44 -> 4.90 mm
- net Net-(D113-DOUT): track 21.9 -> 25.0 mm
- net Net-(D83-A): track 3.25 -> 6.02 mm
- net Net-(D88-A): track 3.25 -> 5.97 mm
- net Net-(D79-A): track 3.24 -> 5.90 mm
- net Net-(D81-A): track 3.24 -> 5.90 mm
- net Net-(D80-A): track 3.24 -> 5.90 mm
- net Net-(D73-A): track 3.26 -> 5.92 mm
- net Net-(D78-A): track 3.24 -> 5.90 mm
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- added copper zone on F.Cu, net GND
