File: hardware/rp_voyager.kicad_pcb (KiCad board)
At the start: 4 copper layers, 150.5 x 141.7 mm, 316 parts, among them J1 INPUT USB, J2 UART USB, J3 INPUT USB, J4 UART USB, Q1 2N7002, SW1 RESET, SW10 Key, SW11 Key, SW12 Key, SW13 Key, SW14 Key, SW15 Key, SW16 Key, SW17 Key, SW18 Key, SW19 Key, SW2 BOOTSEL, SW20 Key, SW21 Key, SW22 Key, SW23 Key, SW24 Key, SW25 Key, SW26 Key, SW27 Key, SW28 Key, SW29 RotaryEncoder_Switch_MP, SW3 Key, SW30 RESET, SW31 BOOTSEL, SW32 Key, SW33 Key, SW34 Key, SW35 Key, SW36 Key, SW37 Key, SW38 Key, SW39 Key, SW4 Key, SW40 Key, SW41 Key, SW42 Key, SW43 Key, SW44 Key, SW45 Key, SW46 Key, SW47 Key, SW48 Key, SW49 Key, SW5 Key, SW50 Key, SW51 Key, SW52 Key, SW53 Key, SW54 Key, SW55 Key, SW56 Key, SW57 Key, SW58 RotaryEncoder_Switch_MP, SW6 Key, SW7 Key, SW8 Key, SW9 Key, U1 TPS259261, U2 AP2125N-3.3TRG1, U3 RP2354A, U4 74HCT1G125GW, U5 TPS259261, U6 AP2125N-3.3TRG1, U7 RP2354A, U8 74HCT1G125GW, Y1 12MHz, Y2 12MHz

Commit message: flip 5v bulk caps on right panel
so no traces go on the edges
Parts:
- moved C67 3.38 mm to (246.7, 92.9), turned to 0 degrees
- moved C71 3.38 mm to (246.8, 90.7), turned to 0 degrees
- moved C69 0.79 mm to (262.2, 51.3)
- moved C65 0.79 mm to (260.1, 51.2)
- turned C66 to 0 degrees
- turned C70 to 0 degrees
Routing:
- net Net-(D89-DIN): track 76.2 -> 84.8 mm, vias 3 -> 1
- net /Right/Connector and Power/+5V: track 635.0 -> 642.9 mm, vias 51 -> 53
- net /Right/Key Matrix (copy)/ROW0: track 178.6 -> 181.4 mm
- net /Right/Key Matrix (copy)/ROW1: track 163.2 -> 160.5 mm

Commit message: fix key switch Kailh Choc v2 compat
Parts:
- moved C28 17.5 mm to (151.8, 51.2), turned to 90 degrees
- moved C32 13.7 mm to (154.8, 51.1), turned to 90 degrees
- moved C31 5.16 mm to (167.0, 111.7)
- moved R12 4.37 mm to (147.2, 106.8)
- moved C35 4.15 mm to (167.0, 109.6)
- moved C29 4.05 mm to (167.7, 74.2)
- moved C33 4.05 mm to (167.5, 71.2)
- moved C30 3.94 mm to (167.4, 93.2)
- moved C34 3.94 mm to (167.3, 90.3)
- moved R13 2.21 mm to (147.2, 104.9)
Routing:
- net /Right/Encoder (copy)/SW_COL: track 195.3 -> 176.9 mm, vias 2 -> 4
- net /Right/Key Matrix (copy)/COL5: track 139.5 -> 135.7 mm
- net Net-(R12-Pad2): track 1.90 -> 5.42 mm
- net /Left/Connector and Power/+5V: track 666.2 -> 663.1 mm, vias 53 -> 52
- net Net-(D93-DOUT): track 23.3 -> 26.2 mm
- net GND: track 256.4 -> 254.0 mm, vias 265 -> 261
- net /Right/Connector and Power/+5V: track 642.9 -> 640.9 mm
- net Net-(U7-~{QSPI_SS}): track 46.2 -> 44.3 mm
- net Net-(R13-Pad2): track 1.80 -> 3.67 mm
- net Net-(U3-~{QSPI_SS}): track 43.1 -> 45.0 mm
- net Net-(D32-DOUT): track 22.7 -> 24.3 mm
- net Net-(U3-RUN): track 40.0 -> 41.1 mm
- net Net-(D102-DOUT): track 29.9 -> 31.0 mm
- net Net-(D31-DIN): track 74.8 -> 74.0 mm
- net Net-(D106-DIN): track 31.8 -> 31.0 mm
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Other:
- board text added: "${TITLE} ${REVISION} at ${ISSUE_DATE} by ${COMPANY}"
