File: hardware/rp_voyager.kicad_pcb (KiCad board)
At the start: 4 copper layers, 150.5 x 141.7 mm, 316 parts, among them J1 INPUT USB, J2 UART USB, J3 INPUT USB, J4 UART USB, Q1 2N7002, SW1 RESET, SW10 Key, SW11 Key, SW12 Key, SW13 Key, SW14 Key, SW15 Key, SW16 Key, SW17 Key, SW18 Key, SW19 Key, SW2 BOOTSEL, SW20 Key, SW21 Key, SW22 Key, SW23 Key, SW24 Key, SW25 Key, SW26 Key, SW27 Key, SW28 Key, SW29 RotaryEncoder_Switch_MP, SW3 Key, SW30 RESET, SW31 BOOTSEL, SW32 Key, SW33 Key, SW34 Key, SW35 Key, SW36 Key, SW37 Key, SW38 Key, SW39 Key, SW4 Key, SW40 Key, SW41 Key, SW42 Key, SW43 Key, SW44 Key, SW45 Key, SW46 Key, SW47 Key, SW48 Key, SW49 Key, SW5 Key, SW50 Key, SW51 Key, SW52 Key, SW53 Key, SW54 Key, SW55 Key, SW56 Key, SW57 Key, SW58 RotaryEncoder_Switch_MP, SW6 Key, SW7 Key, SW8 Key, SW9 Key, U1 TPS259261, U2 AP2125N-3.3TRG1, U3 RP2354A, U4 74HCT1G125GW, U5 TPS259261, U6 AP2125N-3.3TRG1, U7 RP2354A, U8 74HCT1G125GW, Y1 12MHz, Y2 12MHz

Commit message: release v1.1
Parts:
- added R42: 1M, PCM_Resistor_SMD_AKL:R_0603_1608Metric, B.Cu at (245.2, 103.6)
- moved C26 0.15 mm to (171.1, 106.7)
Routing:
- net Net-(D92-DOUT): track 50.1 -> 58.6 mm
- net Net-(U7-~{QSPI_SS}): track 44.3 -> 48.7 mm, vias 4 -> 2
- net /Left/Key Matrix/ROW3: track 155.4 -> 151.1 mm
- net /Right/Encoder (copy)/SW_COL: track 176.8 -> 179.0 mm, vias 4 -> 2
- net /Right/Key Matrix (copy)/COL4: track 147.6 -> 149.4 mm
- net /Right/Key Matrix (copy)/COL1: track 162.9 -> 164.6 mm, vias 4 -> 2
- net /Right/Key Matrix (copy)/ROW3: track 140.4 -> 138.9 mm, vias 4 -> 0
- net /Right/Key Matrix (copy)/ROW2: track 157.8 -> 156.4 mm, vias 4 -> 2
- net /Right/Key Matrix (copy)/COL0: track 185.4 -> 184.1 mm
- net GND: track 238.8 -> 239.9 mm, vias 251 -> 252
- net Net-(Q1-G): track 3.24 -> 4.20 mm
- net /Right/Key Matrix (copy)/COL2: track 146.3 -> 145.4 mm, vias 2 -> 0
- net /Right/Key Matrix (copy)/COL5: track 134.4 -> 133.6 mm, vias 2 -> 1
- net /Left/Connector and Power/CONN_TX: track 14.7 -> 15.4 mm
- net Net-(D89-DIN): track 84.6 -> 85.2 mm, vias 1 -> 3
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
Commit message: PCB: right side layout should match left side
Parts:
- moved D88 0.38 mm to (243.4, 163.2)
- moved D93 0.38 mm to (235.6, 158.7)
- moved SW57 0.38 mm to (238.2, 163.2)
- moved D83 0.37 mm to (257.6, 149.6)
- moved D98 0.37 mm to (249.8, 145.1)
- moved SW52 0.37 mm to (252.4, 149.6)
- moved D101 0.31 mm to (291.8, 86.6)
- moved D102 0.31 mm to (291.8, 105.6)
- moved D106 0.31 mm to (310.9, 110.4)
- moved D66 0.31 mm to (353.5, 123.0)
- moved D70 0.31 mm to (334.4, 123.0)
- moved D72 0.31 mm to (315.4, 80.1)
- moved D74 0.31 mm to (315.4, 118.3)
- moved D76 0.31 mm to (296.3, 75.4)
- moved D77 0.31 mm to (296.3, 94.4)
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Routing:
- net /Right/Connector and Power/+5V: track 641.1 -> 647.7 mm
- net GND: track 239.9 -> 235.1 mm
- net /Right/Key Matrix (copy)/COL1: track 164.6 -> 169.4 mm
- net /Right/Key Matrix (copy)/COL2: track 145.4 -> 150.1 mm
- net /Right/Key Matrix (copy)/COL0: track 184.1 -> 188.2 mm
- net /Right/Encoder (copy)/SW_COL: track 179.0 -> 182.6 mm
- net /Right/Key Matrix (copy)/COL5: track 133.6 -> 137.1 mm
- net /Right/Key Matrix (copy)/COL4: track 149.4 -> 151.5 mm
- net Net-(D113-DOUT): track 25.0 -> 23.0 mm
- net Net-(D101-DOUT): track 21.5 -> 20.4 mm
- net /Right/Key Matrix (copy)/ROW0: track 181.2 -> 180.2 mm
- net Net-(D92-DIN): track 36.5 -> 37.3 mm
- net Net-(D103-DOUT): track 21.1 -> 20.4 mm
- net Net-(D104-DIN): track 31.7 -> 31.0 mm
- net /Right/Key Matrix (copy)/ROW2: track 156.4 -> 155.8 mm
