File: hardware/backlight.kicad_sch (KiCad schematic)
At the start: 39 parts, among them U4 74HCT1G125GW

Commit message: crystal placement, bulk C, wiring updates
Parts:
- C26: footprint PCM_Capacitor_SMD_Handsoldering_AKL:C_1210_3225Metric -> PCM_Capacitor_Tantalum_SMD_Handsoldering_AKL:CP_EIA-3528-21_Kemet-B; symbol Device:C_Small -> Device:C_Polarized_Small
Changed lines of the file:
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@@
 		(title "Voyager keyboard with RP235x")
 		(date "2026-05-17")
-		(rev "0")
+		(rev "1x")
 		(company "Julian7")
 		(comment 1 "RGB backlight")
@@
 	)
 	(symbol
-		(lib_id "Device:C_Small")
+		(lib_id "Device:C_Polarized_Small")
 		(at 67.31 81.28 0)
 		(unit 1)
@@
 		(fields_autoplaced yes)
 		(property "Reference" "C26"
-			(at 69.85 80.0162 0)
+			(at 69.85 79.4638 0)
 			(show_name no)
 			(do_not_autoplace no)
@@
 		)
 		(property "Value" "220u"
-			(at 69.85 82.5562 0)
+			(at 69.85 82.0038 0)
 			(show_name no)
 			(do_not_autoplace no)
@@
 			)
 		)
-		(property "Footprint" "PCM_Capacitor_SMD_Handsoldering_AKL:C_1210_3225Metric"
+		(property "Footprint" "PCM_Capacitor_Tantalum_SMD_Handsoldering_AKL:CP_EIA-3528-21_Kemet-B"
 			(at 67.31 81.28 0)
 			(hide yes)
@@
 			)
 		)
-		(property "Description" "220uF 6.3V Polymer"
+		(property "Description" "Polarized capacitor, small symbol"
 			(at 67.31 81.28 0)
 			(hide yes)
