File: hardware/rp2354a.kicad_sch (KiCad schematic)
At the start: 26 parts, among them SW1 RESET, SW2 BOOTSEL, U3 RP2354A, Y1 12MHz

Commit message: crystal placement, bulk C, wiring updates
Parts:
- Y1: footprint PCM_Crystal_AKL:Crystal_SMD_3225-4Pin_3.2x2.5mm_HandSoldering -> PCM_Crystal_AKL:Crystal_SMD_Abracon_ABM8G-4Pin_3.2x2.5mm
Changed lines of the file:
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@@
 		(title "Voyager keyboard with RP235x")
 		(date "2026-05-17")
-		(rev "0")
+		(rev "1x")
 		(company "Julian7")
 		(comment 1 "RP2354A MCU")
@@
 	)
 	(no_connect
+		(at 140.97 146.05)
+	)
+	(no_connect
 		(at 140.97 143.51)
-	)
-	(no_connect
-		(at 140.97 146.05)
 	)
 	(no_connect
@@
 			)
 		)
-		(property "Footprint" "PCM_Crystal_AKL:Crystal_SMD_3225-4Pin_3.2x2.5mm_HandSoldering"
+		(property "Footprint" "PCM_Crystal_AKL:Crystal_SMD_Abracon_ABM8G-4Pin_3.2x2.5mm"
 			(at 88.9 132.08 0)
 			(hide yes)
