File: hardware/usbc_right.kicad_sch (KiCad schematic)
At the start: 35 parts, among them J3 INPUT USB, J4 UART USB, Q1 2N7002, U5 TPS259261, U6 AP2125N-3.3TRG1

Commit message: make the pcb compatible with kailh choc v1/v2
Parts:
- R29: footprint PCM_Resistor_SMD_AKL:R_1206_3216Metric -> rp_voyager:R_1206_3216Metric_WireJumper
Changed lines of the file:
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@@
 			)
 		)
-		(property "Footprint" "PCM_Resistor_SMD_AKL:R_1206_3216Metric"
+		(property "Footprint" "rp_voyager:R_1206_3216Metric_WireJumper"
 			(at 173.99 121.92 0)
 			(hide yes)
@@
 		(exclude_from_sim no)
 		(in_bom no)
-		(on_board yes)
+		(on_board no)
 		(in_pos_files yes)
 		(dnp no)

Commit message: crystal placement, bulk C, wiring updates
Parts:
- C44: footprint PCM_Capacitor_SMD_Handsoldering_AKL:C_1210_3225Metric -> PCM_Capacitor_Tantalum_SMD_Handsoldering_AKL:CP_EIA-3528-21_Kemet-B; symbol Device:C_Small -> Device:C_Polarized_Small
Changed lines of the file:
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@@
 		(title "Voyager keyboard with RP235x")
 		(date "2026-05-17")
-		(rev "0")
+		(rev "1x")
 		(company "Julian7")
 		(comment 1 "Power supply and UART connector")
@@
 	)
 	(symbol
-		(lib_id "Device:C_Small")
+		(lib_id "Device:C_Polarized_Small")
 		(at 220.98 58.42 0)
 		(unit 1)
@@
 		(fields_autoplaced yes)
 		(property "Reference" "C44"
-			(at 223.52 57.1562 0)
+			(at 223.52 56.6038 0)
 			(show_name no)
 			(do_not_autoplace no)
@@
 		)
 		(property "Value" "220u"
-			(at 223.52 59.6962 0)
+			(at 223.52 59.1438 0)
 			(show_name no)
 			(do_not_autoplace no)
@@
 			)
 		)
-		(property "Footprint" "PCM_Capacitor_SMD_Handsoldering_AKL:C_1210_3225Metric"
+		(property "Footprint" "PCM_Capacitor_Tantalum_SMD_Handsoldering_AKL:CP_EIA-3528-21_Kemet-B"
 			(at 220.98 58.42 0)
 			(hide yes)
@@
 			)
 		)
-		(property "Description" "220uF 6.3V Polymer"
+		(property "Description" "Polarized capacitor, small symbol"
 			(at 220.98 58.42 0)
 			(hide yes)

Commit message: release v1.1
Parts:
- added R42: 1M, PCM_Resistor_SMD_AKL:R_0603_1608Metric, symbol Device:R_Small
Connections:
- net GND: now also R42.2
- net at Q1.1 (G), R30.2: now also R42.1
Other:
- moved on the sheet: Q1
